Commit message: modify abot geometric feature

File: abot_description/urdf/abot_with_rplidar.urdf.xacro (robot description, xacro)
@@ -3,5 +3,5 @@
 	<xacro:include filename="$(find abot_description)/urdf/abot_body.urdf.xacro" />
 	<xacro:include filename="$(find abot_description)/urdf/rplidar.xacro" />
-	<xacro:property name="rplidar_offset_x" value="0" />
+	<xacro:property name="rplidar_offset_x" value="0.021" />
 	<xacro:property name="rplidar_offset_y" value="0" />
 	<xacro:property name="rplidar_offset_z" value="0.028" />
