Commit message: add nav & teleop

File: abot_description/urdf/abot_body.urdf.xacro (robot description, xacro)
@@ -4,6 +4,6 @@
     <xacro:property name="wheel_radius" value="0.033"/>
     <xacro:property name="wheel_length" value="0.017"/>
-    <xacro:property name="base_link_radius" value="0.13"/>
-    <xacro:property name="base_link_length" value="0.005"/>
+    <xacro:property name="base_link_radius" value="0.1025"/>
+    <xacro:property name="base_link_length" value="0.003"/>
     <xacro:property name="motor_radius" value="0.02"/>
     <xacro:property name="motor_length" value="0.08"/>

Commit message: modify chassis size

File: abot_description/urdf/abot_body.urdf.xacro (robot description, xacro)
@@ -2,15 +2,15 @@
 <robot xmlns:xacro="http://www.ros.org/wiki/xacro">
     <xacro:property name="M_PI" value="3.14159"/>
-    <xacro:property name="wheel_radius" value="0.033"/>
-    <xacro:property name="wheel_length" value="0.017"/>
+    <xacro:property name="wheel_radius" value="0.0325"/>
+    <xacro:property name="wheel_length" value="0.027"/>
     <xacro:property name="base_link_radius" value="0.1025"/>
     <xacro:property name="base_link_length" value="0.003"/>
     <xacro:property name="motor_radius" value="0.02"/>
-    <xacro:property name="motor_length" value="0.08"/>
-    <xacro:property name="motor_x" value="-0.055"/>
-    <xacro:property name="motor_y" value="0.075"/>
-    <xacro:property name="plate_height" value="0.07"/>
-    <xacro:property name="standoff_x" value="0.12"/>
-    <xacro:property name="standoff_y" value="0.10"/>
+    <xacro:property name="motor_length" value="0.06"/>
+    <xacro:property name="motor_x" value="-0.0385"/>
+    <xacro:property name="motor_y" value="0.034"/>
+    <xacro:property name="plate_height" value="0.043"/>
+    <xacro:property name="standoff_x" value="0.08"/>
+    <xacro:property name="standoff_y" value="0.06"/>
     <!-- 定义abot本体的宏 -->
     <xacro:macro name="abot_standoff_2in" params="parent number x_loc y_loc z_loc">
@@ -31,5 +31,5 @@
                 <origin xyz=" 0 0 0 " rpy="0 0 0" />
                 <geometry>
-                    <box size="0.01 0.01 0.07" />
+                    <box size="0.01 0.01 ${plate_height}" />
                 </geometry>
                 <material name="black">
@@ -88,5 +88,5 @@
         </link>
         <joint name="base_footprint_joint" type="fixed">
-            <origin xyz="0 0 ${wheel_radius}" rpy="0 0 0" />
+            <origin xyz="0 0 ${wheel_radius*2}" rpy="0 0 0" />
             <parent link="base_footprint"/>
             <child link="base_link" />
@@ -114,5 +114,5 @@
         </link>
         <joint name="base_left_motor_joint" type="fixed">
-            <origin xyz="${motor_x} ${motor_y} 0" rpy="0 0 0" />
+            <origin xyz="${motor_x} ${motor_y} -${wheel_radius}" rpy="0 0 0" />
             <parent link="base_link"/>
             <child link="left_motor" />
@@ -169,5 +169,5 @@
         </link>
         <joint name="base_right_motor_joint" type="fixed">
-            <origin xyz="${motor_x} -${motor_y} 0" rpy="0 0 0" />
+            <origin xyz="${motor_x} -${motor_y} -${wheel_radius}" rpy="0 0 0" />
             <parent link="base_link"/>
             <child link="right_motor" />
@@ -212,5 +212,5 @@
                 <origin xyz="0 0 0" rpy="${M_PI/2} 0 0"/>
                 <geometry>
-                    <sphere radius="${wheel_radius/2}" />
+                    <sphere radius="${wheel_radius}" />
                 </geometry>
                 <material name="black" />
@@ -219,10 +219,10 @@
                 <origin xyz="0 0 0.01" rpy="${M_PI/2} 0 0" />
                 <geometry>
-                    <sphere radius="${wheel_radius/2}" />
+                    <sphere radius="${wheel_radius}" />
                 </geometry>
             </collision>
         </link>
         <joint name="front_caster_joint" type="fixed">
-            <origin xyz="${base_link_radius-wheel_radius/2} 0 -${wheel_radius/2}" rpy="0 0 0"/>
+            <origin xyz="${base_link_radius-wheel_radius} 0 -${wheel_radius}" rpy="0 0 0"/>
             <parent link="base_link"/>
             <child link="front_caster_link"/>
@@ -258,34 +258,4 @@
             </collision>
         </link>
-        <xacro:abot_standoff_2in parent="standoff_2in_1_link" number="5" x_loc="0" y_loc="0" z_loc="${plate_height}"/>
-        <xacro:abot_standoff_2in parent="standoff_2in_2_link" number="6" x_loc="0" y_loc="0" z_loc="${plate_height}"/>
-        <xacro:abot_standoff_2in parent="standoff_2in_3_link" number="7" x_loc="0" y_loc="0" z_loc="${plate_height}"/>
-        <xacro:abot_standoff_2in parent="standoff_2in_4_link" number="8" x_loc="0" y_loc="0" z_loc="${plate_height}"/>
-        <joint name="plate_2_joint" type="fixed">
-            <origin xyz="0 0 ${plate_height}" rpy="0 0 0" />
-            <parent link="plate_1_link"/>
-            <child link="plate_2_link" />
-        </joint>
-        <link name="plate_2_link">
-            <inertial>
-                <mass value="0.01" />
-                <origin xyz="0 0 0" />
-                <inertia ixx="0.001" ixy="0.0" ixz="0.0"
-                         iyy="0.001" iyz="0.0" izz="0.001" />
-            </inertial>
-            <visual>
-                <origin xyz=" 0 0 0 " rpy="0 0 0" />
-                <geometry>
-                    <cylinder length="${base_link_length}" radius="${base_link_radius}"/>
-                </geometry>
-                <material name="yellow" />
-            </visual>
-            <collision>
-                <origin xyz="0.0 0.0 0.0" rpy="0 0 0" />
-                <geometry>
-                    <cylinder length="${base_link_length}" radius="${base_link_radius}"/>
-                </geometry>
-            </collision>
-        </link>
     </xacro:macro>
 </robot>

File: abot_description/urdf/abot_with_rplidar.urdf.xacro (robot description, xacro)
@@ -11,5 +11,5 @@
 	<joint name="rplidar_joint" type="fixed">
 		<origin xyz="${rplidar_offset_x} ${rplidar_offset_y} ${rplidar_offset_z}" rpy="0 0 0" />
-		<parent link="plate_2_link"/>
+		<parent link="plate_1_link"/>
 		<child link="laser_link"/>
 	</joint>

Commit message: base_link -> base_footprint

File: abot_description/urdf/abot_body.urdf.xacro (robot description, xacro)
@@ -88,5 +88,5 @@
         </link>
         <joint name="base_footprint_joint" type="fixed">
-            <origin xyz="0 0 ${wheel_radius*2}" rpy="0 0 0" />
+            <origin xyz="${-motor_x} 0 ${wheel_radius*2}" rpy="0 0 0" />
             <parent link="base_footprint"/>
             <child link="base_link" />
@@ -114,5 +114,5 @@
         </link>
         <joint name="base_left_motor_joint" type="fixed">
-            <origin xyz="${motor_x} ${motor_y} -${wheel_radius}" rpy="0 0 0" />
+            <origin xyz="${motor_x} ${motor_y} ${-wheel_radius}" rpy="0 0 0" />
             <parent link="base_link"/>
             <child link="left_motor" />
@@ -169,5 +169,5 @@
         </link>
         <joint name="base_right_motor_joint" type="fixed">
-            <origin xyz="${motor_x} -${motor_y} -${wheel_radius}" rpy="0 0 0" />
+            <origin xyz="${motor_x} ${-motor_y} ${-wheel_radius}" rpy="0 0 0" />
             <parent link="base_link"/>
             <child link="right_motor" />
@@ -197,5 +197,5 @@
         </link>
         <joint name="right_wheel_joint" type="continuous">
-            <origin xyz="0 -${(motor_length+wheel_length)/2} 0" rpy="0 0 0"/>
+            <origin xyz="0 ${-(motor_length+wheel_length)/2} 0" rpy="0 0 0"/>
             <parent link="right_motor"/>
             <child link="right_wheel_link"/>
@@ -224,11 +224,11 @@
         </link>
         <joint name="front_caster_joint" type="fixed">
-            <origin xyz="${base_link_radius-wheel_radius} 0 -${wheel_radius}" rpy="0 0 0"/>
+            <origin xyz="${base_link_radius-wheel_radius} 0 ${-wheel_radius}" rpy="0 0 0"/>
             <parent link="base_link"/>
             <child link="front_caster_link"/>
         </joint>
-        <xacro:abot_standoff_2in parent="base_link" number="1" x_loc="-${standoff_x/2 + 0.03}" y_loc="-${standoff_y - 0.03}" z_loc="${plate_height/2}"/>
-        <xacro:abot_standoff_2in parent="base_link" number="2" x_loc="-${standoff_x/2 + 0.03}" y_loc="${standoff_y - 0.03}" z_loc="${plate_height/2}"/>
-        <xacro:abot_standoff_2in parent="base_link" number="3" x_loc="${standoff_x/2}" y_loc="-${standoff_y}" z_loc="${plate_height/2}"/>
+        <xacro:abot_standoff_2in parent="base_link" number="1" x_loc="${-standoff_x/2 - 0.03}" y_loc="${-standoff_y + 0.03}" z_loc="${plate_height/2}"/>
+        <xacro:abot_standoff_2in parent="base_link" number="2" x_loc="${-standoff_x/2 - 0.03}" y_loc="${standoff_y - 0.03}" z_loc="${plate_height/2}"/>
+        <xacro:abot_standoff_2in parent="base_link" number="3" x_loc="${standoff_x/2}" y_loc="${-standoff_y}" z_loc="${plate_height/2}"/>
         <xacro:abot_standoff_2in parent="base_link" number="4" x_loc="${standoff_x/2}" y_loc="${standoff_y}" z_loc="${plate_height/2}"/>
         <joint name="plate_1_joint" type="fixed">

Commit message: add imu_link

File: abot_description/urdf/abot_body.urdf.xacro (robot description, xacro)
@@ -92,4 +92,30 @@
             <child link="base_link" />
         </joint>
+        <link name="imu_link">
+            <inertial>
+                <origin xyz="0.0 0 0"/>
+                <mass value="0.1" />
+                <inertia ixx="0.001" ixy="0.0" ixz="0.0"
+                         iyy="0.001" iyz="0.0" izz="0.001" />
+            </inertial>
+            <visual>
+                <origin xyz="0 0 0" rpy="$0 0 0" />
+                <geometry>
+                    <cylinder radius="0.01" length = "0.01"/>
+                </geometry>
+                <material name="gray" />
+            </visual>
+            <collision>
+                <origin xyz="0 0 0" rpy="$0 0 0" />
+                <geometry>
+                    <cylinder radius="$0.01" length = "$0.01"/>
+                </geometry>
+            </collision>
+        </link>
+        <joint name="base_imu_joint" type="fixed">
+            <origin xyz="$-0.0885 0 0.0065" rpy="0 0 0" />
+            <parent link="base_link"/>
+            <child link="laser_link" />
+        </joint>
         <link name="left_motor">
             <inertial>

Commit message: fix bugs in imu_link

File: abot_description/urdf/abot_body.urdf.xacro (robot description, xacro)
@@ -100,5 +100,5 @@
             </inertial>
             <visual>
-                <origin xyz="0 0 0" rpy="$0 0 0" />
+                <origin xyz="0 0 0" rpy="0 0 0" />
                 <geometry>
                     <cylinder radius="0.01" length = "0.01"/>
@@ -107,12 +107,12 @@
             </visual>
             <collision>
-                <origin xyz="0 0 0" rpy="$0 0 0" />
-                <geometry>
-                    <cylinder radius="$0.01" length = "$0.01"/>
+                <origin xyz="0 0 0" rpy="0 0 0" />
+                <geometry>
+                    <cylinder radius="0.01" length = "0.01"/>
                 </geometry>
             </collision>
         </link>
         <joint name="base_imu_joint" type="fixed">
-            <origin xyz="$-0.0885 0 0.0065" rpy="0 0 0" />
+            <origin xyz="-0.0885 0 0.0065" rpy="0 0 0" />
             <parent link="base_link"/>
             <child link="laser_link" />

Commit message: fix bugs in base_imu_joint

File: abot_description/urdf/abot_body.urdf.xacro (robot description, xacro)
@@ -116,5 +116,5 @@
             <origin xyz="-0.0885 0 0.0065" rpy="0 0 0" />
             <parent link="base_link"/>
-            <child link="laser_link" />
+            <child link="imu_link" />
         </joint>
         <link name="left_motor">
